File: for_enraged_rabbit/easy_optical/easy_optical_pcb/easy_optical_pcb.kicad_pcb (KiCad board)
At the start: 2 copper layers, 10 x 34 mm, 11 parts, among them J1 Conn_01x03, Q1 AO3402_N_Mosfet, U1 ITR20403

Commit message: add more projects
Parts:
- moved R3 0.20 mm to (105.9, 126.6)
Routing:
- net VCC: track 30.8 -> 31.5 mm

Commit message: add 28mm servo selector Version2
Parts:
- R1: value 1k -> 750
Changed lines of the file:
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@@
 			)
 		)
-		(property "Value" "1k"
+		(property "Value" "750"
 			(at 2.7 0 90)
 			(layer "F.Fab")
